File: kicad/side.kicad_sch (KiCad schematic)
At the start: 105 parts, among them J1 AudioJack4_SwitchTR1, Q1 Q_PMOS_GSD, Q3 Q_PMOS_GSD, SW1 SW_Push, SW13 SW_Push, SW14 SW_Push, SW15 SW_Push, SW16 SW_Push, SW17 SW_Push, SW18 SW_Push, SW2 SW_Push, SW25 SW_Push, SW26 SW_Push, SW27 SW_Push, SW28 SW_Push, SW29 SW_Push, SW3 SW_Push, SW30 SW_Push, SW37 SW_Push, SW38 SW_Push, SW39 SW_Push, SW4 SW_Push, SW40 SW_Push, SW41 SW_Push, SW42 SW_Push, SW49 SW_Push, SW5 SW_Push, SW50 SW_Push, SW51 SW_Push, SW52 SW_Push, SW57 SW_SPDT, SW6 SW_Push, U3 XIAO-ESP32-S3-SMD

Commit message: Rerouted PCB
Parts:
- D100: renamed from D94; footprint Library:SK6812MINI-E -> Library:SK6812MINI-E_1-REV
- D101: renamed from D95; footprint Library:SK6812MINI-E -> Library:SK6812MINI-E_1-REV
- D102: renamed from D96; footprint Library:SK6812MINI-E -> Library:SK6812MINI-E_1-REV
- D103: renamed from D97; footprint Library:SK6812MINI-E -> Library:SK6812MINI-E_1-REV
- D104: renamed from D98; footprint Library:SK6812MINI-E -> Library:SK6812MINI-E_1-REV
- D109: renamed from D105; footprint Library:SK6812MINI-E -> Library:SK6812MINI-E_1-REV
- D110: renamed from D106; footprint Library:SK6812MINI-E -> Library:SK6812MINI-E_1-REV
- D111: renamed from D107; footprint Library:SK6812MINI-E -> Library:SK6812MINI-E_1-REV
- D112: renamed from D108; footprint Library:SK6812MINI-E -> Library:SK6812MINI-E_1-REV
- D63: renamed from D57; footprint Library:SK6812MINI-E -> Library:SK6812MINI-E_1-REV
- D64: renamed from D58; footprint Library:SK6812MINI-E -> Library:SK6812MINI-E_1-REV
- D65: renamed from D59; footprint Library:SK6812MINI-E -> Library:SK6812MINI-E_1-REV
- D66: renamed from D60; footprint Library:SK6812MINI-E -> Library:SK6812MINI-E_1-REV
- D67: renamed from D61; footprint Library:SK6812MINI-E -> Library:SK6812MINI-E_1-REV
- D68: renamed from D62; footprint Library:SK6812MINI-E -> Library:SK6812MINI-E_1-REV
- D75: renamed from D69; footprint Library:SK6812MINI-E -> Library:SK6812MINI-E_1-REV
- D76: renamed from D70; footprint Library:SK6812MINI-E -> Library:SK6812MINI-E_1-REV
- D77: renamed from D71; footprint Library:SK6812MINI-E -> Library:SK6812MINI-E_1-REV
- D78: renamed from D72; footprint Library:SK6812MINI-E -> Library:SK6812MINI-E_1-REV
- D79: renamed from D73; footprint Library:SK6812MINI-E -> Library:SK6812MINI-E_1-REV
- D80: renamed from D74; footprint Library:SK6812MINI-E -> Library:SK6812MINI-E_1-REV
- D87: renamed from D81; footprint Library:SK6812MINI-E -> Library:SK6812MINI-E_1-REV
- D88: renamed from D82; footprint Library:SK6812MINI-E -> Library:SK6812MINI-E_1-REV
- D89: renamed from D83; footprint Library:SK6812MINI-E -> Library:SK6812MINI-E_1-REV
- D90: renamed from D84; footprint Library:SK6812MINI-E -> Library:SK6812MINI-E_1-REV
- D91: renamed from D85; footprint Library:SK6812MINI-E -> Library:SK6812MINI-E_1-REV
- D92: renamed from D86; footprint Library:SK6812MINI-E -> Library:SK6812MINI-E_1-REV
- D99: renamed from D93; footprint Library:SK6812MINI-E -> Library:SK6812MINI-E_1-REV
- SW10: renamed from SW4; footprint PCM_marbastlib-xp-gateron_lp:SW_KS33_HS_KS-2P02B01-02_HS_1u -> Library:SW_KS33_HS_KS-2P02B01-02_HS_1u
- SW11: renamed from SW5; footprint PCM_marbastlib-xp-gateron_lp:SW_KS33_HS_KS-2P02B01-02_HS_1u -> Library:SW_KS33_HS_KS-2P02B01-02_HS_1u
- SW12: renamed from SW6; footprint PCM_marbastlib-xp-gateron_lp:SW_KS33_HS_KS-2P02B01-02_HS_1u -> Library:SW_KS33_HS_KS-2P02B01-02_HS_1u
- SW19: renamed from SW13; footprint PCM_marbastlib-xp-gateron_lp:SW_KS33_HS_KS-2P02B01-02_HS_1u -> Library:SW_KS33_HS_KS-2P02B01-02_HS_1u
- SW20: renamed from SW14; footprint PCM_marbastlib-xp-gateron_lp:SW_KS33_HS_KS-2P02B01-02_HS_1u -> Library:SW_KS33_HS_KS-2P02B01-02_HS_1u
- SW21: renamed from SW15; footprint PCM_marbastlib-xp-gateron_lp:SW_KS33_HS_KS-2P02B01-02_HS_1u -> Library:SW_KS33_HS_KS-2P02B01-02_HS_1u
- SW22: renamed from SW16; footprint PCM_marbastlib-xp-gateron_lp:SW_KS33_HS_KS-2P02B01-02_HS_1u -> Library:SW_KS33_HS_KS-2P02B01-02_HS_1u
- SW23: renamed from SW17; footprint PCM_marbastlib-xp-gateron_lp:SW_KS33_HS_KS-2P02B01-02_HS_1u -> Library:SW_KS33_HS_KS-2P02B01-02_HS_1u
- SW24: renamed from SW18; footprint PCM_marbastlib-xp-gateron_lp:SW_KS33_HS_KS-2P02B01-02_HS_1u -> Library:SW_KS33_HS_KS-2P02B01-02_HS_1u
- SW31: renamed from SW25; footprint PCM_marbastlib-xp-gateron_lp:SW_KS33_HS_KS-2P02B01-02_HS_1u -> Library:SW_KS33_HS_KS-2P02B01-02_HS_1u
- SW32: renamed from SW26; footprint PCM_marbastlib-xp-gateron_lp:SW_KS33_HS_KS-2P02B01-02_HS_1u -> Library:SW_KS33_HS_KS-2P02B01-02_HS_1u
- SW33: renamed from SW27; footprint PCM_marbastlib-xp-gateron_lp:SW_KS33_HS_KS-2P02B01-02_HS_1u -> Library:SW_KS33_HS_KS-2P02B01-02_HS_1u
- SW34: renamed from SW28; footprint PCM_marbastlib-xp-gateron_lp:SW_KS33_HS_KS-2P02B01-02_HS_1u -> Library:SW_KS33_HS_KS-2P02B01-02_HS_1u
- SW35: renamed from SW29; footprint PCM_marbastlib-xp-gateron_lp:SW_KS33_HS_KS-2P02B01-02_HS_1u -> Library:SW_KS33_HS_KS-2P02B01-02_HS_1u
- SW36: renamed from SW30; footprint PCM_marbastlib-xp-gateron_lp:SW_KS33_HS_KS-2P02B01-02_HS_1u -> Library:SW_KS33_HS_KS-2P02B01-02_HS_1u
- SW43: renamed from SW37; footprint PCM_marbastlib-xp-gateron_lp:SW_KS33_HS_KS-2P02B01-02_HS_1u -> Library:SW_KS33_HS_KS-2P02B01-02_HS_1u
- SW44: renamed from SW38; footprint PCM_marbastlib-xp-gateron_lp:SW_KS33_HS_KS-2P02B01-02_HS_1u -> Library:SW_KS33_HS_KS-2P02B01-02_HS_1u
- SW45: renamed from SW39; footprint PCM_marbastlib-xp-gateron_lp:SW_KS33_HS_KS-2P02B01-02_HS_1u -> Library:SW_KS33_HS_KS-2P02B01-02_HS_1u
- SW46: renamed from SW40; footprint PCM_marbastlib-xp-gateron_lp:SW_KS33_HS_KS-2P02B01-02_HS_1u -> Library:SW_KS33_HS_KS-2P02B01-02_HS_1u
- SW47: renamed from SW41; footprint PCM_marbastlib-xp-gateron_lp:SW_KS33_HS_KS-2P02B01-02_HS_1u -> Library:SW_KS33_HS_KS-2P02B01-02_HS_1u
- SW48: renamed from SW42; footprint PCM_marbastlib-xp-gateron_lp:SW_KS33_HS_KS-2P02B01-02_HS_1u -> Library:SW_KS33_HS_KS-2P02B01-02_HS_1u
- SW53: renamed from SW49; footprint PCM_marbastlib-xp-gateron_lp:SW_KS33_HS_KS-2P02B01-02_HS_1u -> Library:SW_KS33_HS_KS-2P02B01-02_HS_1u
- SW54: renamed from SW50; footprint PCM_marbastlib-xp-gateron_lp:SW_KS33_HS_KS-2P02B01-02_HS_1u -> Library:SW_KS33_HS_KS-2P02B01-02_HS_1u
- SW55: renamed from SW51; footprint PCM_marbastlib-xp-gateron_lp:SW_KS33_HS_KS-2P02B01-02_HS_1u -> Library:SW_KS33_HS_KS-2P02B01-02_HS_1u
- SW56: renamed from SW52; footprint PCM_marbastlib-xp-gateron_lp:SW_KS33_HS_KS-2P02B01-02_HS_1u -> Library:SW_KS33_HS_KS-2P02B01-02_HS_1u
- SW7: renamed from SW1; footprint PCM_marbastlib-xp-gateron_lp:SW_KS33_HS_KS-2P02B01-02_HS_1u -> Library:SW_KS33_HS_KS-2P02B01-02_HS_1u
- SW8: renamed from SW2; footprint PCM_marbastlib-xp-gateron_lp:SW_KS33_HS_KS-2P02B01-02_HS_1u -> Library:SW_KS33_HS_KS-2P02B01-02_HS_1u
- SW9: renamed from SW3; footprint PCM_marbastlib-xp-gateron_lp:SW_KS33_HS_KS-2P02B01-02_HS_1u -> Library:SW_KS33_HS_KS-2P02B01-02_HS_1u
- renumbered C1 to C2, D4 to D10, D5 to D11, D113 to D114, D6 to D12, D13 to D19, D14 to D20, D15 to D21, D16 to D22, D17 to D23, D18 to D24, D25 to D31, D26 to D32, D27 to D33, D28 to D34, D29 to D35, D30 to D36, D37 to D43, D38 to D44, D39 to D45, D40 to D46, D41 to D47, D42 to D48, D49 to D53, D50 to D54, D51 to D55, D52 to D56, D1 to D7, D2 to D8, D3 to D9, H2 to H10, H3 to H11, H4 to H12, H5 to H13, H6 to H14, H7 to H15, H8 to H16, H1 to H9, J1 to J2, Q1 to Q2, Q3 to Q4, R8 to R10, R1 to R2, R3 to R4, R5 to R6, R7 to R9, SW57 to SW58, TP1 to TP2
Connections:
- net COL3: now also U3.11 (GPIO9_A10_D10_MOSI)
- net COL4: now also U3.10 (GPIO8_A9_D9_MISO)
- net COL5: now also U3.9 (GPIO7_A8_D8_SCK)
- net LED: now also U3.22 (MTCK)
- net LED_EN: now also U3.21 (MTMS)
- net ROW0: now also U3.8 (GPIO44_D7_RX)
- net ROW1: now also U3.7 (GPIO43_A6_D6_TX)
- net ROW2: now also U3.6 (GPIO6_A5_D5_SCL)
- net ROW3: now also U3.5 (GPIO5_A4_D4_SDA)
- net ROW4: now also U3.4 (GPIO4_A3_D3)
- no-connect marks 6 -> 9
Other:
- moved on the sheet: C2, D100, D101, D102, D103, D104, D109, D110, D111, D112, D114, D63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
