File: kicad/split-keyboard.kicad_pcb (KiCad board)
At the start: 2 copper layers, 301.5 x 122.1 mm, 218 parts, among them J1 AudioJack4_SwitchTR1, J2 AudioJack4_SwitchTR1, Q1 Q_PMOS_GSD, Q2 Q_PMOS_GSD, Q3 Q_PMOS_GSD, Q4 Q_PMOS_GSD, SW1 SW_Push, SW10 SW_Push, SW11 SW_Push, SW12 SW_Push, SW13 SW_Push, SW14 SW_Push, SW15 SW_Push, SW16 SW_Push, SW17 SW_Push, SW18 SW_Push, SW19 SW_Push, SW2 SW_Push, SW20 SW_Push, SW21 SW_Push, SW22 SW_Push, SW23 SW_Push, SW24 SW_Push, SW25 SW_Push, SW26 SW_Push, SW27 SW_Push, SW28 SW_Push, SW29 SW_Push, SW3 SW_Push, SW30 SW_Push, SW31 SW_Push, SW32 SW_Push, SW33 SW_Push, SW34 SW_Push, SW35 SW_Push, SW36 SW_Push, SW37 SW_Push, SW38 SW_Push, SW39 SW_Push, SW4 SW_Push, SW40 SW_Push, SW41 SW_Push, SW42 SW_Push, SW43 SW_Push, SW44 SW_Push, SW45 SW_Push, SW46 SW_Push, SW47 SW_Push, SW48 SW_Push, SW49 SW_Push, SW5 SW_Push, SW50 SW_Push, SW51 SW_Push, SW52 SW_Push, SW53 SW_Push, SW54 SW_Push, SW55 SW_Push, SW56 SW_Push, SW57 SW_SPDT, SW58 SW_SPDT, SW6 SW_Push, SW7 SW_Push, SW8 SW_Push, SW9 SW_Push, U3 XIAO-ESP32-S3-SMD, U4 XIAO-ESP32-S3-SMD

Commit message: Rerouted PCB
Parts:
- removed C1: 100 uF, Capacitor_SMD:C_1206_3216Metric
- removed D1, D13, D14, D15, D16, D17, D18, D2, D25, D26, D27, D28, D29, D3, D30, D37, D38, D39, D4, D40, D41, D42, D49, D5, D50, D51, D52, D6: D, Diode_SMD:D_SOD-123
- removed D105, D106, D107, D108, D57, D58, D59, D60, D61, D62, D69, D70, D71, D72, D73, D74, D81, D82, D83, D84, D85, D86, D93, D94, D95, D96, D97, D98: SK6812MINI, Library:SK6812MINI-E
- removed D113: MSE1PG, Diode_SMD:D_MicroSMP_AK
- removed H1, H2, H3, H4, H5, H6, H7, H8: MountingHole, MountingHole:MountingHole_2.2mm_M2
- removed J1: AudioJack4_SwitchTR1, Library:LSH-3956D
- removed Q1, Q3: Q_PMOS_GSD, Package_TO_SOT_SMD:SOT-23
- removed R1: 390, Resistor_SMD:R_0603_1608Metric
- removed R3, R5, R7, R8: 10k, Resistor_SMD:R_1206_3216Metric
- removed REF** (x6): MouseBite-Slot_2.0x4.5mm_outset_D0.5mm_P0.85mm_7h, Panelization:MouseBite-Slot_2.0x4.5mm_outset_D0.5mm_P0.85mm_7h
- removed SW1, SW13, SW14, SW15, SW16, SW17, SW18, SW2, SW25, SW26, SW27, SW28, SW29, SW3, SW30, SW37, SW38, SW39, SW4, SW40, SW41, SW42, SW49, SW5, SW50, SW51, SW52, SW6: SW_Push, PCM_marbastlib-xp-gateron_lp:SW_KS33_HS_KS-2P02B01-02_HS_1u
- removed SW57: SW_SPDT, Library:SK12D07VG5
- removed TP1: BAT, Connector_JST:JST_PH_S2B-PH-K_1x02_P2.00mm_Horizontal
- D100, D101, D102, D103, D104, D109, D110, D111, D112, D63, D64, D65, D66, D67, D68, D75, D76, D77, D78, D79, D80, D87, D88, D89, D90, D91, D92, D99: footprint Library:SK6812MINI-E -> Library:SK6812MINI-E_1-REV
- D114, G***, Q4, R10, R9: moved to B.Cu
- SW10, SW11, SW12, SW19, SW20, SW21, SW22, SW23, SW24, SW31, SW32, SW33, SW34, SW35, SW36, SW43, SW44, SW45, SW46, SW47, SW48, SW53, SW54, SW55, SW56, SW7, SW8, SW9: footprint PCM_marbastlib-xp-gateron_lp:SW_KS33_HS_KS-2P02B01-02_HS_1u -> Library:SW_KS33_HS_KS-2P02B01-02_HS_1u
- U3: moved to F.Cu
- moved U3 191.8 mm to (151.0, 147.4), turned to 0 degrees
- moved G*** 172.3 mm to (179.5, 176.0), turned to 180 degrees
- moved G*** 113.4 mm to (173.2, 175.3)
- moved D114 90.0 mm to (139.4, 155.3), turned to 90 degrees
- moved R10 89.0 mm to (139.2, 151.3), turned to 90 degrees
- moved R9 87.1 mm to (136.7, 160.7), turned to 112.5 degrees
- moved Q4 86.6 mm to (136.4, 156.4)
- moved R4 83.3 mm to (140.1, 159.2)
- moved Q2 82.8 mm to (139.7, 162.5), turned to -157.5 degrees
- moved R6 82.1 mm to (139.9, 166.7), turned to -67.5 degrees
- moved H9 81.6 mm to (182.0, 132.8)
- moved TP2 80.9 mm to (144.8, 160.4)
- moved D104 80.5 mm to (267.6, 156.2)
- moved D68 80.5 mm to (267.6, 99.0)
- moved D80 80.5 mm to (267.6, 118.1)
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Connections:
- U3 pad 1: /left/COL0 -> /right/COL0
- U3 pad 10: /left/ROW3 -> /right/COL4
- U3 pad 11: /left/ROW4 -> /right/COL3
- U3 pad 15: /left/VBAT -> /right/VBAT
- U3 pad 17: /left/IO 1 -> /right/IO 1
- U3 pad 18: /left/IO 2 -> /right/IO 2
- U3 pad 19: /left/EN -> /right/EN
- U3 pad 2: /left/COL1 -> /right/COL1
- U3 pad 21: /left/LED -> /right/LED_EN
- U3 pad 22: /left/LED_EN -> /right/LED
- U3 pad 3: /left/COL2 -> /right/COL2
- U3 pad 4: /left/COL3 -> /right/ROW4
- U3 pad 5: /left/COL4 -> /right/ROW3
- U3 pad 6: /left/COL5 -> /right/ROW2
- U3 pad 7: /left/ROW0 -> /right/ROW1
- U3 pad 8: /left/ROW1 -> /right/ROW0
- U3 pad 9: /left/ROW2 -> /right/COL5
Routing:
- net /left/VLED: track 788.0 -> 0.00 mm, vias 6 -> 0
- net /left/COL5: track 250.0 -> 0.00 mm, vias 1 -> 0
- net /left/COL4: track 230.1 -> 0.00 mm, vias 1 -> 0
- net /left/COL3: track 211.1 -> 0.00 mm, vias 1 -> 0
- net /left/COL2: track 188.5 -> 0.00 mm, vias 1 -> 0
- net /left/ROW0: track 168.3 -> 0.00 mm
- net /left/COL1: track 162.4 -> 0.00 mm, vias 1 -> 0
- net /left/ROW3: track 147.0 -> 0.00 mm
- net /left/ROW1: track 132.0 -> 0.00 mm
- net /left/ROW2: track 128.1 -> 0.00 mm
- net /left/COL0: track 122.7 -> 0.00 mm, vias 1 -> 0
- net /left/ROW4: track 115.4 -> 0.00 mm
- net /left/EN: track 58.5 -> 0.00 mm
- net /left/LED: track 55.6 -> 0.00 mm, vias 2 -> 0
- net /left/LED_EN: track 37.1 -> 0.00 mm
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Other:
- board size 301.5 x 122.1 mm -> 149.8 x 122.1 mm
