File: kicad/split-keyboard.kicad_sch (KiCad schematic)
At the start: 0 parts

Commit message: Rerouted PCB
Other:
- removed sheet left
Changed lines of the file:
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@@
-		)
-	)
-	(sheet
-		(at 113.03 62.23)
-		(size 41.91 27.94)
-		(exclude_from_sim no)
-		(in_bom yes)
-		(on_board yes)
-		(dnp no)
-		(fields_autoplaced yes)
-		(stroke
-			(width 0.1524)
-			(type solid)
-		)
-		(fill
-			(color 0 0 0 0.0000)
-		)
-		(property "Sheetname" "left"
-			(at 113.03 61.5184 0)
-			(effects
-				(font
-					(size 1.27 1.27)
-				)
-				(justify left bottom)
-			)
-		)
-		(property "Sheetfile" "side.kicad_sch"
-			(at 113.03 90.7546 0)
-			(effects
-				(font
-					(size 1.27 1.27)
-				)
-				(justify left top)
-			)
-		)
-		(instances
-			(project "split-keyboard"
-				(path "/0a2fdc8f-22d7-408a-9ed7-1983688b8147"
-					(page "2")
-				)
-			)
 		)
 	)
